File: Micromod/MicroMod_Processor_Board.kicad_sch (KiCad schematic)
At the start: 3 parts, among them J1 MICROMOD-2222, U1 STM32H747XIHx

Commit message: add the stm32h5 with all connections to schematic
Parts:
- removed U1: STM32H747XIHx, Package_BGA:TFBGA-265_14x14mm_Layout17x17_P0.8mm, symbol MCU_ST_STM32H7:STM32H747XIHx
- added C1: 1u, symbol Device:C
- added C10, C18: 2.2uF, symbol Device:C
- added C11, C12, C13, C14, C15, C16, C17: 100n, symbol Device:C_Small
- added C2, C3: 6.8pF, symbol Device:C
- added C4, C7, C9: 100n, symbol Device:C
- added C5: 4.7uF, symbol Device:C
- added C6: 10uF, symbol Device:C
- added C8: 1uF, symbol Device:C
- added D1: ESDA6V1-5SC6, Package_TO_SOT_SMD:SOT-23-6, symbol Power_Protection:ESDA6V1-5SC6
- added F1: 0.2A, symbol Device:Fuse
- added J2: Micro_SD_Card, symbol Connector:Micro_SD_Card
- added J3: WiFi_BT_CONN_2, symbol Connector_Generic:Conn_02x10_Odd_Even
- added J4: WiFi_BT_CONN_1, symbol Connector_Generic:Conn_02x10_Odd_Even
- added J5: TRACE, symbol Connector_Generic:Conn_02x10_Odd_Even
- added Q1: FDN340P, Package_TO_SOT_SMD:SOT-23, symbol Transistor_FET:FDN340P
- added R1: R, symbol Device:R
- added R2: 100k, symbol Device:R
- added R3: DNP, symbol Device:R
- added U1: STM32H562VGTx, Package_QFP:LQFP-100_14x14mm_P0.5mm, symbol MCU_ST_STM32H5:STM32H562VGTx
- added Y1: ABS07AIG-32.768KHZ, symbol Device:Crystal
Connections:
- net +3.3V: now also C7.2, C8.2, F1.1, J2.4 (VDD), J3.1 (Pin_1), J3.2 (Pin_2), J4.1 (Pin_1), J4.2 (Pin_2), Q1.2 (S), R1.1, U1.21 (VREF+)
- net A0: now also U1.35 (PB0)
- net A1: now also U1.36 (PB1)
- net AUD_BCLK: now also U1.30 (PA5)
- net AUD_IN-CAM_PCLK: now also U1.31 (PA6)
- net AUD_LRCLK: now also U1.29 (PA4)
- net AUD_MCLK: now also U1.33 (PC4)
- net AUD_OUT-CAM_MCLK: now also U1.32 (PA7)
- net BATT_VIN: now also U1.15 (PC0)
- net CAN-RX: now also U1.81 (PD0)
- net CAN-TX: now also U1.82 (PD1)
- net D0: now also U1.23 (PA0)
- net D1-CAM_TRIG: now also U1.24 (PA1)
- net G11-SWO: now also J5.6 (Pin_6), R3.2
- net G3: now also U1.18 (PC3)
- net G4: now also U1.57 (PD10)
- net G6: now also J5.8 (Pin_8), U1.77 (PA15(JTDI))
- net G7: now also U1.84 (PD3)
- net G8: now also U1.85 (PD4)
- net G9-CAM_HSYNC: now also U1.86 (PD5)
- net GND: now also C1.2, C10.2, C11.1, C12.1, C13.1, C14.1, C15.1, C16.1, C17.1, C18.2, C2.2, C3.2, C4.2, C5.2, C6.2, C7.1, C8.1, C9.2, J2.6 (VSS), J2.9 (SHIELD), J3.13 (Pin_13), J3.14 (Pin_14), J3.19 (Pin_19), J3.20 (Pin_20), J3.6 (Pin_6), J3.7 (Pin_7), J4.10 (Pin_10), J4.13 (Pin_13), J4.14 (Pin_14), J4.17 (Pin_17), J4.18 (Pin_18), J4.19 (Pin_19), J4.20 (Pin_20), J4.3 (Pin_3), J4.4 (Pin_4), J4.8 (Pin_8), J4.9 (Pin_9), J5.15 (Pin_15), J5.17 (Pin_17), J5.19 (Pin_19), J5.3 (Pin_3), J5.5 (Pin_5), R2.2, U1.10 (VSS), U1.19 (VSSA), U1.20 (VREF-), U1.27 (VSS), U1.49 (VSS), U1.7 (PC13), U1.74 (VSS), U1.99 (VSS)
- net I2C_SCL: now also U1.92 (PB6)
- net I2C_SCL1: now also U1.95 (PB8)
- net I2C_SDA: now also U1.93 (PB7)
- net I2C_SDA1: now also U1.96 (PB9)
- net I2C_~{INT}: now also U1.91 (PB5)
- net PWM0: now also U1.69 (PA10)
- net PWM1: now also U1.67 (PA8)
- net SDIO_CMD-SPI_COPI1: now also U1.45 (PE14)
- net SDIO_DATA0-SPI_CIPO1: now also U1.44 (PE13)
- net SDIO_DATA1: now also U1.97 (PE0)
- net SDIO_DATA2: now also U1.46 (PE15)
- net SDIO_DATA3-~{SPI_CS1}: now also U1.42 (PE11)
- net SDIO_SCK-SPI_SCK1: now also U1.43 (PE12)
- net SPI_CIPO-LED_CLK: now also U1.17 (PC2)
- net SPI_COPI-LED_DAT: now also U1.16 (PC1)
- net SPI_SCK: now also U1.47 (PB10)
- net SWDCK: now also J5.4 (Pin_4), U1.76 (PA14(JTCK)
- net SWDIO: now also J5.2 (Pin_2), U1.72 (PA13(JTMS)
- net UART_CTS1: now also U1.52 (PB13)
- net UART_RTS1: now also U1.59 (PD12)
- net UART_RX1: now also U1.56 (PD9)
- net UART_RX2: now also U1.64 (PC7)
- net UART_TX1: now also U1.55 (PD8)
- net UART_TX2: now also U1.63 (PC6)
- net USB_D+: now also U1.71 (PA12)
- net USB_D-: now also U1.70 (PA11)
- net ~{BOOT}: now also Q1.1 (G), R1.2
- net ~{RESET}: now also C9.1, J5.10 (Pin_10), U1.14 (NRST)
- net ~{SPI_CS}: now also U1.51 (PB12)
- net RTC_3V_BATT renamed VBAT
- net VBAT: now also C1.1, U1.6 (VBAT)
- net USBHOST_D+: no longer names the net of J1.35 (USBHOST_D+)
- net USBHOST_D-: no longer names the net of J1.37 (USBHOST_D-)
- new net: C3.1, U1.9 (PC15), Y1.1
- new net: C18.1, U1.48 (VCAP)
- new net: C12.2, C13.2, C14.2, C15.2, C16.2, C17.2, U1.100 (VDD), U1.11 (VDD), U1.22 (VDDA), U1.28 (VDD), U1.50 (VDD), U1.75 (VDD)
- new net: C2.1, U1.8 (PC14), Y1.2
- new net: C10.1, U1.98 (VCAP)
- new net BOOT0: Q1.3 (D), R2.1, U1.94 (BOOT0)
- new net BT_DEV_WAKE: J3.11 (Pin_11), U1.62 (PD15)
- new net BT_HOST_WAKE: J3.4 (Pin_4), U1.25 (PA2)
- new net BT_PCM_CLK: J3.18 (Pin_18), U1.58 (PD11)
- new net BT_PCM_IN: J3.15 (Pin_15), U1.26 (PA3)
- new net BT_PCM_OUT: J3.17 (Pin_17), U1.37 (PB2)
- new net BT_PCM_SYNC: J3.16 (Pin_16), U1.34 (PC5)
- new net BT_REG_ON: J3.3 (Pin_3), U1.60 (PD13)
- new net BT_UART_CTS: J3.8 (Pin_8), U1.41 (PE10)
- new net BT_UART_RTS: J3.10 (Pin_10), U1.40 (PE9)
- new net BT_UART_RX: J3.9 (Pin_9), U1.39 (PE8)
- new net BT_UART_TX: J3.5 (Pin_5), U1.38 (PE7)
- new net MCU_VCC: C11.2, C4.1, C5.1, C6.1, F1.2, J5.1 (Pin_1), U1.73 (VDDUSB)
- new net SD_CLK: J2.5 (CLK), U1.87 (PD6)
- new net SD_CMD: J2.3 (CMD), U1.88 (PD7)
- new net SD_DAT0: J2.7 (DAT0), U1.53 (PB14)
- new net SD_DAT1: J2.8 (DAT1), U1.54 (PB15)
- new net SD_DAT2: J2.1 (DAT2), U1.89 (PB3(JTDO)
- new net SD_DAT3: J2.2 (DAT3/CD), R3.1, U1.90 (PB4(NJTRST))
- new net TRACE_CLK: J5.12 (Pin_12), U1.1 (PE2)
- new net TRACE_D0: J5.14 (Pin_14), U1.2 (PE3)
- new net TRACE_D1: J5.16 (Pin_16), U1.3 (PE4)
- new net TRACE_D2: J5.18 (Pin_18), U1.4 (PE5)
- new net TRACE_D3: J5.20 (Pin_20), U1.5 (PE6)
- new net WIFI_SDIO_CLK: J4.7 (Pin_7), U1.80 (PC12)
- new net WIFI_SDIO_CMD: J4.5 (Pin_5), U1.83 (PD2)
- new net WIFI_SDIO_DAT0: J4.15 (Pin_15), U1.65 (PC8)
- new net WIFI_SDIO_DAT1: J4.11 (Pin_11), U1.66 (PC9)
- new net WIFI_SDIO_DAT2: J4.12 (Pin_12), U1.78 (PC10)
- new net WIFI_SDIO_DAT3: J4.16 (Pin_16), U1.79 (PC11)
- new net WL_GPIO_0_HOST_WAKE: J4.6 (Pin_6), U1.68 (PA9)
- new net WL_REG_ON: J3.12 (Pin_12), U1.61 (PD14)
- no-connect marks 0 -> 8

Commit message: progress so far
Parts:
- C1, C10, C11, C12, C13, C14, C15, C16, C17, C18, C2, C3, C4, C5, C6, C7, C8, C9: footprint (none) -> Capacitor_SMD:C_0603_1608Metric_Pad1.08x0.95mm_HandSolder
- F1: footprint (none) -> Resistor_SMD:R_0805_2012Metric_Pad1.20x1.40mm_HandSolder
- J2: footprint (none) -> Connector_Card:microSD_HC_Wuerth_693072010801
- J3, J4: footprint (none) -> Library:CONN20_DF40HC-25-20DS_HIR
- J5: footprint (none) -> Connector_PinHeader_1.27mm:PinHeader_2x10_P1.27mm_Vertical_SMD
- R1, R2, R3: footprint (none) -> Resistor_SMD:R_0603_1608Metric_Pad0.98x0.95mm_HandSolder
- Y1: footprint (none) -> Resistor_SMD:R_1206_3216Metric_Pad1.30x1.75mm_HandSolder
Connections:
- net +3.3V: now also C11.2, C12.2, C13.2, C14.2, C15.2, C16.2, C17.2, C4.1, C5.1, C6.1, J5.1 (Pin_1), U1.100 (VDD), U1.11 (VDD), U1.22 (VDDA), U1.28 (VDD), U1.50 (VDD), U1.73 (VDDUSB), U1.75 (VDD); no longer J1.2 (3.3V), J1.74 (3.3V)
- net BT_PCM_CLK: now also J3.15 (Pin_15); no longer J3.18 (Pin_18)
- net BT_PCM_IN: now also J3.16 (Pin_16); no longer J3.15 (Pin_15)
- net BT_PCM_OUT: now also J3.18 (Pin_18); no longer J3.17 (Pin_17)
- net BT_PCM_SYNC: now also J3.17 (Pin_17); no longer J3.16 (Pin_16)
- net BT_UART_CTS: now also J3.5 (Pin_5); no longer J3.8 (Pin_8)
- net BT_UART_RTS: now also J3.8 (Pin_8); no longer J3.10 (Pin_10)
- net BT_UART_TX: now also J3.10 (Pin_10); no longer J3.5 (Pin_5)
- net G0: now also U1.86 (PD5)
- net G1: now also U1.97 (PE0)
- net G2: now also U1.46 (PE15)
- net G5: now also U1.85 (PD4)
- net GND: no longer J4.18 (Pin_18), J4.20 (Pin_20)
- net WIFI_SDIO_CLK: now also J4.18 (Pin_18); no longer J4.7 (Pin_7)
- net WIFI_SDIO_CMD: now also J4.20 (Pin_20); no longer J4.5 (Pin_5)
- net WIFI_SDIO_DAT0: now also J4.11 (Pin_11); no longer J4.15 (Pin_15)
- net WIFI_SDIO_DAT1: now also J4.15 (Pin_15); no longer J4.11 (Pin_11)
- net G10-CAM_VSYNC: no longer names the net of J1.63 (G10/ADC_D+/CAM_VSYNC)
- net G8: no longer names the net of J1.67 (G8)
- net G8: no longer U1.85 (PD4)
- net G9-CAM_HSYNC: no longer names the net of J1.65 (G9/ADC_D-/CAM_HSYNC)
- net G9-CAM_HSYNC: no longer U1.86 (PD5)
- removed net MCU_VCC: C11.2, C4.1, C5.1, C6.1, F1.2, J5.1 (Pin_1), U1.73 (VDDUSB)
- net SDIO_CMD-SPI_COPI1 renamed SPI_COPI1
- net SDIO_DATA0-SPI_CIPO1 renamed SPI_CIPO1
- net SDIO_DATA1: no longer names the net of J1.66 (SDIO_DATA1)
- net SDIO_DATA1: no longer U1.97 (PE0)
- net SDIO_DATA2: no longer names the net of J1.68 (SDIO_DATA2)
- net SDIO_DATA2: no longer U1.46 (PE15)
- net SDIO_DATA3-~{SPI_CS1} renamed ~{SPI_CS1}
- net SDIO_SCK-SPI_SCK1 renamed SPI_SCK1
- net SPI_CIPO-LED_CLK renamed SPI_MISO
- net SPI_COPI-LED_DAT renamed SPI_MOSI
- new net: F1.2, J1.2 (3.3V), J1.74 (3.3V)
- no-connect marks 8 -> 13
Other:
- note added: "SDMMC1_D0(PC8, AF12): WIFI_SDIO_DAT0 SDMMC1_D1(PC9, AF12): WIFI_SDIO_DAT1 SDMMC1_D2(PC10, AF12): WIFI_SDIO_DAT2 SDMMC1_D3(PC11, AF12): WIFI_SDIO_DAT3 SDMMC1_CLK(PC12, AF12): WIFI_SDIO_CLK SDMMC1_CMD(PD2, AF12): WIFI_SDIO_CMD SDMMC2_D0(PB14, AF9): SD_DAT0 SDMMC2_D1(PB15, AF9): SD_DAT1 SDMMC2_D2(PB3, AF9): SD_DAT2 SDMMC2_D3(PB4, AF9): SD_DAT3 SDMMC2_CLK(PD6, AF11): SD_CLK SDMMC2_CMD(PD7, AF11): SD_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"
- note added: "USART6_TX(PC6, AF7): UART_TX2 USART6_RX(PC7, AF7): UART_RX2 USART3_TX(PD8, AF7): UART_TX1 USART3_RX(PD9, AF7): UART_RX1 USART3_RTS(PD12, AF7): UART_RTS1 USART3_CTS(PB13, AF7): UART_CTS1 USART7_RX(PE7, AF7): BT_UART_TX USART7_TX(PE8, AF7): BT_UART_RX USART7_RTS(PE9, AF7): BT_UART_RTS USART7_CTS(PE10, AF7): BT_UART_CTS I2C1_SCL(PB7, AF4): I2C_SCL I2C1_SDA(PB6, AF4): I2C_SDA I2C1_INT(PB5, GPIO): I2C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"
- moved on the sheet: F1, J5

Commit message: almost done routing
Parts:
- removed D1: ESDA6V1-5SC6, Package_TO_SOT_SMD:SOT-23-6, symbol Power_Protection:ESDA6V1-5SC6
Connections:
- net BT_DEV_WAKE: now also U1.46 (PE15); no longer U1.62 (PD15)
- net BT_REG_ON: now also U1.24 (PA1); no longer U1.60 (PD13)
- net D1-CAM_TRIG: now also U1.85 (PD4); no longer U1.24 (PA1)
- net G1: now also U1.77 (PA15(JTDI)); no longer U1.97 (PE0)
- net G2: now also U1.69 (PA10); no longer U1.46 (PE15)
- net G3: now also U1.68 (PA9); no longer U1.18 (PC3)
- net G5: now also U1.60 (PD13); no longer U1.85 (PD4)
- net G6: now also U1.61 (PD14); no longer J5.8 (Pin_8), U1.77 (PA15(JTDI))
- net G7: now also U1.62 (PD15); no longer U1.84 (PD3)
- net PWM0: now also U1.18 (PC3); no longer J1.32 (PWM0), U1.69 (PA10)
- net PWM1: now also U1.57 (PD10); no longer J1.47 (PWM1), U1.67 (PA8)
- net WL_GPIO_0_HOST_WAKE: now also U1.84 (PD3); no longer U1.68 (PA9)
- net WL_REG_ON: now also U1.51 (PB12); no longer U1.61 (PD14)
- net ~{SPI_CS}: now also U1.67 (PA8); no longer U1.51 (PB12)
- net G4: no longer names the net of J1.48 (G4/BUS4)
- net G4: no longer U1.57 (PD10)
- no-connect marks 13 -> 17

Commit message: done
Parts:
- added D1: LED, LED_SMD:LED_0603_1608Metric_Pad1.05x0.95mm_HandSolder, symbol Device:LED
- added R4: 470, Resistor_SMD:R_0603_1608Metric_Pad0.98x0.95mm_HandSolder, symbol Device:R
- added R5: 1k, Resistor_SMD:R_0603_1608Metric_Pad0.98x0.95mm_HandSolder, symbol Device:R
Connections:
- net GND: now also J4.5 (Pin_5), J4.7 (Pin_7), D1.1 (K)
- net at U1.97 (PE0): now also R4.2
- net 3.3V_EN: no longer names the net of J1.4 (3.3V_EN)
- net PWM0 renamed USB_VIN
- net USB_VIN: now also R5.1
- net PWM1: no longer names the net of U1.57 (PD10)
- net V_USB: no longer names the net of J1.9 (USB_VIN)
- net V_USB: now also R5.2
- new net: D1.2 (A), R4.1
- no-connect marks 17 -> 19

Commit message: add some changes, make ibom from both pcbs
Parts:
- R1: value R -> 100k
- U1: value STM32H562VGTx -> STM32H563VGTx

Commit message: fix the rts/cts line being swapped and missing led0 connection (PWM0)
Connections:
- net PWM0: now reaches J1.32 (PWM0)
- net PWM0: now also U1.57 (PD10)
- no-connect marks 19 -> 17
